Commit message: World file creatd

File: description/robot.urdf.xacro (robot description, xacro)
@@ -3,3 +3,4 @@
     <xacro:include filename="$(find my_bot)/description/robot_core.xacro"/>
     <!--xacro:include filename="robot_core.xacro" /-->
+    <xacro:include filename="$(find my_bot)/description/gazebo_control.xacro"/>
 </robot>

File: description/robot_core.xacro (robot description, xacro)
@@ -39,4 +39,7 @@
         </xacro:inertial_box>
     </link>
+    <gazebo reference="chassis">
+        <material>Gazebo/White</material>
+    </gazebo>
     <joint name="left_wheel_joint" type="continuous">
         <parent link="base_link"/>
@@ -63,4 +66,7 @@
         </xacro:inertial_cylinder>
     </link>
+    <gazebo reference="left_wheel">
+        <material>Gazebo/Blue</material>
+    </gazebo>
     <joint name="right_wheel_joint" type="continuous">
         <parent link="base_link"/>
@@ -87,3 +93,32 @@
         </xacro:inertial_cylinder>
     </link>
+    <gazebo reference="right_wheel">
+        <material>Gazebo/Blue</material>
+    </gazebo>
+    <joint name="caster_wheel_joint" type="fixed">
+        <parent link="chassis"/>
+        <child link="caster_wheel"/>
+        <origin xyz="0.24 0 0"/>
+    </joint>
+    <link name="caster_wheel">
+        <visual>
+            <geometry>
+                <sphere radius="0.05"/>
+            </geometry>
+            <material name="black"/>
+        </visual>
+        <collision>
+            <geometry>
+                <sphere radius="0.05"/>
+            </geometry>
+        </collision>
+        <xacro:inertial_sphere mass="0.1" radius="0.05">
+            <origin xyz="0 0 0" rpy="0 0 0"/>
+        </xacro:inertial_sphere>
+    </link>
+    <gazebo reference="caster_wheel">
+        <material>Gazebo/Black</material>
+        <mu1 value="0.001"/>
+        <mu2 value="0.001"/>
+    </gazebo>
 </robot>

Commit message: Ros2 control in Gazebo done

File: description/robot.urdf.xacro (robot description, xacro)
@@ -3,4 +3,8 @@
     <xacro:include filename="$(find my_bot)/description/robot_core.xacro"/>
     <!--xacro:include filename="robot_core.xacro" /-->
-    <xacro:include filename="$(find my_bot)/description/gazebo_control.xacro"/>
+    <!--xacro:include filename="$(find my_bot)/description/gazebo_control.xacro"/-->
+    <xacro:include filename="$(find my_bot)/description/ros2_control.xacro"/>
+    <xacro:include filename="$(find my_bot)/description/lidar.xacro"/>
+    <xacro:include filename="$(find my_bot)/description/camera.xacro"/>
+    <!--xacro:include filename="$(find my_bot)/description/depth_camera.xacro"/-->
 </robot>

File: description/robot_core.xacro (robot description, xacro)
@@ -13,4 +13,7 @@
     <material name="black">
         <color rgba="0 0 0 1" />
+    </material>
+    <material name="red">
+        <color rgba="1 0 0 1" />
     </material>
     <link name="base_link">

Commit message: Ros2 control with Gazebo with extra bits done

File: description/robot.urdf.xacro (robot description, xacro)
@@ -1,8 +1,12 @@
 <?xml version="1.0"?>
 <robot xmlns:xacro="http://www.ros.org/wiki/xacro"  name="robot">
+    <xacro:arg name="use_ros2_control" default="true"/>
     <xacro:include filename="$(find my_bot)/description/robot_core.xacro"/>
-    <!--xacro:include filename="robot_core.xacro" /-->
-    <!--xacro:include filename="$(find my_bot)/description/gazebo_control.xacro"/-->
-    <xacro:include filename="$(find my_bot)/description/ros2_control.xacro"/>
+    <xacro:if value="$(arg use_ros2_control)">
+        <xacro:include filename="$(find my_bot)/description/ros2_control.xacro" />
+    </xacro:if>
+    <xacro:unless value="$(arg use_ros2_control)">
+        <xacro:include filename="$(find my_bot)/description/gazebo_control.xacro" />
+    </xacro:unless>
     <xacro:include filename="$(find my_bot)/description/lidar.xacro"/>
     <xacro:include filename="$(find my_bot)/description/camera.xacro"/>

File: description/robot_core.xacro (robot description, xacro)
@@ -62,5 +62,5 @@
             <!--origin xyz="0.15 0 0.075"/-->
             <geometry>
-                <cylinder radius="0.05" length="0.04"/>
+                <sphere radius="0.05"/>
             </geometry>
         </collision>
@@ -89,5 +89,5 @@
             <!--origin xyz="0.15 0 0.075"/-->
             <geometry>
-                <cylinder radius="0.05" length="0.04"/>
+                <sphere radius="0.05"/>
             </geometry>
         </collision>
