Commit message: Final working repo

File: description/lidar.xacro (robot description, xacro)
@@ -8,5 +8,5 @@
     <link name="laser_frame">
         <visual>
-            <!--origin xyz="0.15 0 0.075"/-->
+            <!-- <origin xyz="0.06 0 0"/> -->
             <geometry>
                 <cylinder radius="0.05" length="0.04"/>
@@ -21,5 +21,5 @@
         </collision>
         <xacro:inertial_cylinder mass="0.1" length="0.04" radius="0.05">
-            <origin xyz="0 0 0" rpy="0 0 0"/>
+            <origin xyz="0.1 0 0" rpy="0 0 0"/>
         </xacro:inertial_cylinder>
     </link>

File: description/robot_core.xacro (robot description, xacro)
@@ -52,4 +52,5 @@
         <material>Gazebo/White</material>
     </gazebo>
+    <!--Back wheels-->
     <joint name="left_wheel_joint" type="continuous">
         <parent link="base_link"/>
